File: CPS3-OSCR.kicad_pcb (KiCad board)
At the start: 4 copper layers, 117.6 x 100 mm, 42 parts, among them J1 128MB, J2 64MB, J3 CART SLOT TOP ROW, J4 CART SLOT BOTTOM ROW, J5 5145154-1, J6 Conn_02x03_Counter_Clockwise, J7 Conn_02x03_Counter_Clockwise, M2_1 Screw_Terminal_01x01, M2_2 Screw_Terminal_01x01, M2_3 Screw_Terminal_01x01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

Commit message: Fix 5822030-3 model orientation
Other:
- board text added: "72"
Changed lines of the file:
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@@
 			)
 		)
-		(property "Footprint" "58220303"
+		(property "Footprint" "5822030-3:58220303"
 			(at 0 0 180)
 			(layer "F.Fab")
@@
 		(model "${KIPRJMOD}/../5822030-3/3D/5822030-3.stp"
 			(offset
-				(xyz 47.61999822 -0.6799999969 4.849999832)
+				(xyz 47.619998 -0.68 4.85)
 			)
 			(scale
@@
 			)
 			(rotate
-				(xyz -90 0 0)
+				(xyz -90 0 180)
 			)
 		)
@@
 			)
 		)
-		(property "Footprint" "58220303"
+		(property "Footprint" "5822030-3:58220303"
 			(at 0 0 180)
 			(layer "F.Fab")
@@
 		(model "${KIPRJMOD}/../5822030-3/3D/5822030-3.stp"
 			(offset
-				(xyz 47.61999822 -0.6799999969 4.849999832)
+				(xyz 47.619998 -0.68 4.85)
 			)
 			(scale
@@
 			)
 			(rotate
-				(xyz -90 0 0)
+				(xyz -90 0 180)
 			)
 		)
@@
 		)
 	)
+	(gr_text "72"
+		(at 102.37 120.7631 0)
+		(layer "F.SilkS")
+		(effects
+			(font
+				(size 1 1)
+				(thickness 0.15)
+			)
+		)
+	)
 	(gr_text "0"
 		(at 171.14 85.205 0)
@@
 		)
 	)
+	(gr_text "72"
+		(at 102.37 139.783101 0)
+		(layer "F.SilkS")
+		(effects
+			(font
+				(size 1 1)
+				(thickness 0.15)
+			)
+		)
+	)
 	(gr_text "5"
 		(at 125.42 100.445 0)
@@
 		(layer "F.SilkS")
 		(effects
+			(font
+				(size 1 1)
+				(thickness 0.15)
+			)
+		)
+	)
+	(gr_text "1"
+		(at 197.62 139.783101 0)
+		(layer "F.SilkS")
+		(effects
+			(font
+				(size 1 1)
+				(thickness 0.15)
+			)
+		)
+	)
+	(gr_text "1"
+		(at 197.62 120.7631 0)
+		(layer "F.SilkS")
+		(effects
